Commit message: fix(urdf): rotate base_scan 180° — RPLIDAR C1 angle 0 is at cable side not arrow

File: hardware/urdf/turtlebot3_burger_sensors.urdf.xacro (robot description, xacro)
@@ -253,5 +253,5 @@
     <parent link="base_link"/>
     <child  link="base_scan"/>
-    <origin xyz="-0.032 0.0 0.172" rpy="0 0 0"/>
+    <origin xyz="-0.032 0.0 0.172" rpy="0 0 3.14159"/>
   </joint>
   <link name="base_scan">
